File: ai03-pcb-tutorial.kicad_pcb (KiCad board)
At the start: 2 copper layers, 68.3 x 38.1 mm, 24 parts, among them SW1 SW_Push, U1 ATmega32U4-A, Y1 16MHz

Commit message: Add gerbers
Other:
- outline, holes or cut-outs redrawn
- board text added: "2x2 by dale"
Changed lines of the file:
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@@
     )
   )
-  (gr_line (start 99.21875 112.7125) (end 161.925 112.7125) (layer "Edge.Cuts") (width 0.1))
-  (gr_arc (start 164.30625 148.43125) (mid 163.608798 150.115048) (end 161.925 150.8125) (layer "Edge.Cuts") (width 0.1))
-  (gr_line (start 99.21875 150.8125) (end 161.925 150.8125) (layer "Edge.Cuts") (width 0.1))
+  (gr_line (start 164.30625 150.8125) (end 99.21875 150.8125) (layer "Edge.Cuts") (width 0.1))
   (gr_arc (start 99.21875 150.8125) (mid 96.973686 149.882564) (end 96.04375 147.6375) (layer "Edge.Cuts") (width 0.1))
   (gr_arc (start 96.04375 115.8875) (mid 96.973686 113.642436) (end 99.21875 112.7125) (layer "Edge.Cuts") (width 0.1))
+  (gr_line (start 99.21875 112.7125) (end 164.30625 112.7125) (layer "Edge.Cuts") (width 0.1))
   (gr_line (start 96.04375 115.8875) (end 96.04375 147.6375) (layer "Edge.Cuts") (width 0.1))
-  (gr_arc (start 161.925 112.7125) (mid 163.608798 113.409952) (end 164.30625 115.09375) (layer "Edge.Cuts") (width 0.1))
-  (gr_line (start 164.30625 115.09375) (end 164.30625 148.43125) (layer "Edge.Cuts") (width 0.1))
+  (gr_line (start 164.30625 112.7125) (end 164.30625 150.8125) (layer "Edge.Cuts") (width 0.1))
+  (gr_text "2x2 by dale" (at 116.68125 114.3) (layer "F.SilkS")
+    (effects (font (size 1 1) (thickness 0.15)))
+  )
   (segment (start 121.5875 138.14375) (end 114.30625 138.14375) (width 0.381) (layer "F.Cu") (net 1))
   (segment (start 98.10373 129.54627) (end 99.21875 128.43125) (width 0.381) (layer "F.Cu") (net 1))
